Commit message: update world file & add topic_check code

File: src/turtlebot/turtlebot_description/urdf/bases/create_gazebo.urdf.xacro (robot description, xacro)
@@ -6,6 +6,6 @@
 	    <alwaysOn>true</alwaysOn>
 	    <updateRate>50</updateRate>
-	    <leftJoint>left_wheel_joint</leftJoint>
-    	    <rightJoint>right_wheel_joint</rightJoint>
+	    <leftJoint>right_wheel_joint</leftJoint>
+    	    <rightJoint>left_wheel_joint</rightJoint>
 	    <wheelSeparation>.230</wheelSeparation>
 	    <wheelDiameter>0.070</wheelDiameter>
@@ -25,201 +25,4 @@
 	  </plugin>
 	</gazebo>
-    <gazebo reference="left_wheel_link">
-      <mu1>1.0</mu1>
-      <mu2>1.0</mu2>
-      <kp>1000000.0</kp>
-      <kd>100.0</kd>
-      <minDepth>0.001</minDepth>
-      <maxVel>1.0</maxVel>
-    </gazebo>
-    <gazebo reference="right_wheel_link">
-      <mu1>1.0</mu1>
-      <mu2>1.0</mu2>
-      <kp>1000000.0</kp>
-      <kd>100.0</kd>
-      <minDepth>0.001</minDepth>
-      <maxVel>1.0</maxVel>
-    </gazebo>
-    <gazebo reference="rear_wheel_link">
-      <mu1>0.0</mu1>
-      <mu2>0.0</mu2>
-      <kp>1000000.0</kp>
-      <kd>100.0</kd>
-      <minDepth>0.001</minDepth>
-      <maxVel>1.0</maxVel>
-    </gazebo>
-    <gazebo reference="front_wheel_link">
-      <mu1>0.0</mu1>
-      <mu2>0.0</mu2>
-      <kp>1000000.0</kp>
-      <kd>100.0</kd>
-      <minDepth>0.001</minDepth>
-      <maxVel>1.0</maxVel>
-    </gazebo>
-	</xacro:macro>
-	<xacro:macro name="sim_imu">
-	  <gazebo>
-	    <plugin name="imu_controller" filename="libgazebo_ros_imu.so">
-	      <alwaysOn>true</alwaysOn>
-	      <updateRate>30</updateRate>
-	      <bodyName>gyro_link</bodyName>
-	      <topicName>imu/data</topicName>
-        <serviceName>imu/is_calibrated</serviceName>
-	      <gaussianNoise>${0.0017*0.0017}</gaussianNoise>
-        <xyzOffsets>0 0 0</xyzOffsets>
-        <rpyOffsets>0 0 0</rpyOffsets>
-      </plugin>
-	  </gazebo>
-	</xacro:macro>
-	<xacro:macro name="sim_create_wall_sensor">
-	  <gazebo reference="wall_sensor_link">
-      <sensor type="ray" name="wall_sensor">
-        <always_on>true</always_on>
-        <update_rate>20.0</update_rate>
-        <pose>0 0 0 0 0 0</pose>
-        <visualize>false</visualize>
-        <ray>
-          <scan>
-            <horizontal>
-              <samples>1</samples>
-              <resolution>1</resolution>
-              <min_angle>0</min_angle>
-              <max_angle>0</max_angle>
-            </horizontal>
-          </scan>
-          <range>
-            <min>0.0160</min>
-            <max>0.04</max>
-            <resolution>0.1</resolution>
-          </range>
-        </ray>
-      </sensor>
-	  </gazebo>
-	</xacro:macro>
-	<xacro:macro name="sim_create_cliff_sensors">
-	  <gazebo reference="left_cliff_sensor_link">
-      <sensor type="ray" name="left_cliff_sensor">
-        <always_on>true</always_on>
-        <update_rate>20.0</update_rate>
-        <pose>0 0 0 0 0 0</pose>
-        <visualize>false</visualize>
-        <ray>
-          <scan>
-            <horizontal>
-              <samples>1</samples>
-              <resolution>1</resolution>
-              <min_angle>0</min_angle>
-              <max_angle>0</max_angle>
-            </horizontal>
-          </scan>
-          <range>
-            <min>0.01</min>
-            <max>0.04</max>
-            <resolution>0.1</resolution>
-          </range>
-        </ray>
-      </sensor>
-	  </gazebo>
-	  <gazebo reference="right_cliff_sensor_link">
-      <sensor type="ray" name="right_cliff_sensor">
-        <always_on>true</always_on>
-        <update_rate>20.0</update_rate>
-        <pose>0 0 0 0 0 0</pose>
-        <visualize>false</visualize>
-        <ray>
-          <scan>
-            <horizontal>
-              <samples>1</samples>
-              <resolution>1</resolution>
-              <min_angle>0</min_angle>
-              <max_angle>0</max_angle>
-            </horizontal>
-          </scan>
-          <range>
-            <min>0.01</min>
-            <max>0.04</max>
-            <resolution>0.1</resolution>
-          </range>
-        </ray>
-      </sensor>
-	  </gazebo>
-	  <gazebo reference="leftfront_cliff_sensor_link">
-      <sensor type="ray" name="leftfront_cliff_sensor">
-        <always_on>true</always_on>
-        <update_rate>20.0</update_rate>
-        <pose>0 0 0 0 0 0</pose>
-        <visualize>false</visualize>
-        <ray>
-          <scan>
-            <horizontal>
-              <samples>1</samples>
-              <resolution>1</resolution>
-              <min_angle>0</min_angle>
-              <max_angle>0</max_angle>
-            </horizontal>
-          </scan>
-          <range>
-            <min>0.01</min>
-            <max>0.04</max>
-            <resolution>0.1</resolution>
-          </range>
-        </ray>
-      </sensor>
-	  </gazebo>
-	  <gazebo reference="rightfront_cliff_sensor_link">
-      <sensor type="ray" name="rightfront_cliff_sensor">
-        <always_on>true</always_on>
-        <update_rate>20.0</update_rate>
-        <pose>0 0 0 0 0 0</pose>
-        <visualize>false</visualize>
-        <ray>
-          <scan>
-            <horizontal>
-              <samples>1</samples>
-              <resolution>1</resolution>
-              <min_angle>0</min_angle>
-              <max_angle>0</max_angle>
-            </horizontal>
-          </scan>
-          <range>
-            <min>0.01</min>
-            <max>0.04</max>
-            <resolution>0.1</resolution>
-          </range>
-        </ray>
-      </sensor>
-	  </gazebo>
-<!--
-    <gazebo reference="laser_sensor_link">
-      <sensor type="ray" name="laser_sensor">
-        <pose>0 0 0 0 0 0</pose>
-        <visualize>true</visualize>
-        <update_rate>40</update_rate>
-        <ray>
-          <scan>
-            <horizontal>
-              <samples>720</samples>
-              <resolution>1</resolution>
-              <min_angle>-1.570796</min_angle>
-              <max_angle>1.570796</max_angle>
-            </horizontal>
-          </scan>
-          <range>
-            <min>0.10</min>
-            <max>30.0</max>
-            <resolution>0.01</resolution>
-          </range>
-          <noise>
-            <type>gaussian</type>
-            <mean>0.0</mean>
-            <stddev>0.01</stddev>
-          </noise>
-        </ray>
-        <plugin name="gazebo_ros_head_hokuyo_controller" filename="libgazebo_ros_laser.so">
-          <topicName>/kobuki/laser/scan</topicName>
-          <frameName>laser_sensor_link</frameName>
-        </plugin>
-      </sensor>
-    </gazebo> -->
 <!--
 	  <gazebo>
@@ -238,4 +41,201 @@
 	    </plugin>
 	  </gazebo> -->
+    <gazebo reference="left_wheel_link">
+      <mu1>1.0</mu1>
+      <mu2>1.0</mu2>
+      <kp>1000000.0</kp>
+      <kd>100.0</kd>
+      <minDepth>0.001</minDepth>
+      <maxVel>1.0</maxVel>
+    </gazebo>
+    <gazebo reference="right_wheel_link">
+      <mu1>1.0</mu1>
+      <mu2>1.0</mu2>
+      <kp>1000000.0</kp>
+      <kd>100.0</kd>
+      <minDepth>0.001</minDepth>
+      <maxVel>1.0</maxVel>
+    </gazebo>
+    <gazebo reference="rear_wheel_link">
+      <mu1>0.0</mu1>
+      <mu2>0.0</mu2>
+      <kp>1000000.0</kp>
+      <kd>100.0</kd>
+      <minDepth>0.001</minDepth>
+      <maxVel>1.0</maxVel>
+    </gazebo>
+    <gazebo reference="front_wheel_link">
+      <mu1>0.0</mu1>
+      <mu2>0.0</mu2>
+      <kp>1000000.0</kp>
+      <kd>100.0</kd>
+      <minDepth>0.001</minDepth>
+      <maxVel>1.0</maxVel>
+    </gazebo>
+	</xacro:macro>
+	<xacro:macro name="sim_imu">
+	  <gazebo>
+	    <plugin name="imu_controller" filename="libgazebo_ros_imu.so">
+	      <alwaysOn>true</alwaysOn>
+	      <updateRate>30</updateRate>
+	      <bodyName>gyro_link</bodyName>
+	      <topicName>imu/data</topicName>
+        <serviceName>imu/is_calibrated</serviceName>
+	      <gaussianNoise>${0.0017*0.0017}</gaussianNoise>
+        <xyzOffsets>0 0 0</xyzOffsets>
+        <rpyOffsets>0 0 0</rpyOffsets>
+      </plugin>
+	  </gazebo>
+	</xacro:macro>
+	<xacro:macro name="sim_create_wall_sensor">
+	  <gazebo reference="wall_sensor_link">
+      <sensor type="ray" name="wall_sensor">
+        <always_on>true</always_on>
+        <update_rate>20.0</update_rate>
+        <pose>0 0 0 0 0 0</pose>
+        <visualize>false</visualize>
+        <ray>
+          <scan>
+            <horizontal>
+              <samples>1</samples>
+              <resolution>1</resolution>
+              <min_angle>0</min_angle>
+              <max_angle>0</max_angle>
+            </horizontal>
+          </scan>
+          <range>
+            <min>0.0160</min>
+            <max>0.04</max>
+            <resolution>0.1</resolution>
+          </range>
+        </ray>
+      </sensor>
+	  </gazebo>
+	</xacro:macro>
+	<xacro:macro name="sim_create_cliff_sensors">
+	  <gazebo reference="left_cliff_sensor_link">
+      <sensor type="ray" name="left_cliff_sensor">
+        <always_on>true</always_on>
+        <update_rate>20.0</update_rate>
+        <pose>0 0 0 0 0 0</pose>
+        <visualize>false</visualize>
+        <ray>
+          <scan>
+            <horizontal>
+              <samples>1</samples>
+              <resolution>1</resolution>
+              <min_angle>0</min_angle>
+              <max_angle>0</max_angle>
+            </horizontal>
+          </scan>
+          <range>
+            <min>0.01</min>
+            <max>0.04</max>
+            <resolution>0.1</resolution>
+          </range>
+        </ray>
+      </sensor>
+	  </gazebo>
+	  <gazebo reference="right_cliff_sensor_link">
+      <sensor type="ray" name="right_cliff_sensor">
+        <always_on>true</always_on>
+        <update_rate>20.0</update_rate>
+        <pose>0 0 0 0 0 0</pose>
+        <visualize>false</visualize>
+        <ray>
+          <scan>
+            <horizontal>
+              <samples>1</samples>
+              <resolution>1</resolution>
+              <min_angle>0</min_angle>
+              <max_angle>0</max_angle>
+            </horizontal>
+          </scan>
+          <range>
+            <min>0.01</min>
+            <max>0.04</max>
+            <resolution>0.1</resolution>
+          </range>
+        </ray>
+      </sensor>
+	  </gazebo>
+	  <gazebo reference="leftfront_cliff_sensor_link">
+      <sensor type="ray" name="leftfront_cliff_sensor">
+        <always_on>true</always_on>
+        <update_rate>20.0</update_rate>
+        <pose>0 0 0 0 0 0</pose>
+        <visualize>false</visualize>
+        <ray>
+          <scan>
+            <horizontal>
+              <samples>1</samples>
+              <resolution>1</resolution>
+              <min_angle>0</min_angle>
+              <max_angle>0</max_angle>
+            </horizontal>
+          </scan>
+          <range>
+            <min>0.01</min>
+            <max>0.04</max>
+            <resolution>0.1</resolution>
+          </range>
+        </ray>
+      </sensor>
+	  </gazebo>
+	  <gazebo reference="rightfront_cliff_sensor_link">
+      <sensor type="ray" name="rightfront_cliff_sensor">
+        <always_on>true</always_on>
+        <update_rate>20.0</update_rate>
+        <pose>0 0 0 0 0 0</pose>
+        <visualize>false</visualize>
+        <ray>
+          <scan>
+            <horizontal>
+              <samples>1</samples>
+              <resolution>1</resolution>
+              <min_angle>0</min_angle>
+              <max_angle>0</max_angle>
+            </horizontal>
+          </scan>
+          <range>
+            <min>0.01</min>
+            <max>0.04</max>
+            <resolution>0.1</resolution>
+          </range>
+        </ray>
+      </sensor>
+	  </gazebo>
+<!--
+    <gazebo reference="laser_sensor_link">
+      <sensor type="ray" name="laser_sensor">
+        <pose>0 0 0 0 0 0</pose>
+        <visualize>true</visualize>
+        <update_rate>40</update_rate>
+        <ray>
+          <scan>
+            <horizontal>
+              <samples>720</samples>
+              <resolution>1</resolution>
+              <min_angle>-1.570796</min_angle>
+              <max_angle>1.570796</max_angle>
+            </horizontal>
+          </scan>
+          <range>
+            <min>0.10</min>
+            <max>30.0</max>
+            <resolution>0.01</resolution>
+          </range>
+          <noise>
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