Commit message: update dumper & realsense_sim

File: src/turtlebot/turtlebot_description/urdf/bases/create.urdf.xacro (robot description, xacro)
@@ -64,8 +64,8 @@
 			</geometry>
 			</visual>
-			<collision>
+			<collision name="base_link">
 			<origin xyz="0.0 0.0 0.0308" rpy="0 0 0" />
 			<geometry>
-				<cylinder length="0.0611632" radius="0.16495"/>
+				<cylinder length="0.0611632" radius="0.17"/>
 			</geometry>
 			</collision>
@@ -262,6 +262,6 @@
 	  <!-- Simulation sensors -->
 		<sim_create/>
-		<sim_create_wall_sensor/>
-		<sim_create_cliff_sensors/>
+		<!-- <sim_create_wall_sensor/> -->
+		<!-- <sim_create_cliff_sensors/> -->
 		<sim_imu/>
   	</xacro:macro>

File: src/turtlebot/turtlebot_description/urdf/bases/create_gazebo.urdf.xacro (robot description, xacro)
@@ -120,17 +120,17 @@
         <update_rate>20.0</update_rate>
         <pose>0 0 0 0 0 0</pose>
-        <visualize>false</visualize>
-        <ray>
-          <scan>
-            <horizontal>
-              <samples>1</samples>
-              <resolution>1</resolution>
-              <min_angle>0</min_angle>
-              <max_angle>0</max_angle>
-            </horizontal>
-          </scan>
-          <range>
-            <min>0.01</min>
-            <max>0.04</max>
+        <visualize>true</visualize>
+        <ray>
+          <scan>
+            <horizontal>
+              <samples>720</samples>
+              <resolution>1</resolution>
+              <min_angle>-1.570796</min_angle>
+              <max_angle>1.570796</max_angle>
+            </horizontal>
+          </scan>
+          <range>
+            <min>0.01</min>
+            <max>0.5</max>
             <resolution>0.1</resolution>
           </range>
@@ -143,17 +143,17 @@
         <update_rate>20.0</update_rate>
         <pose>0 0 0 0 0 0</pose>
-        <visualize>false</visualize>
-        <ray>
-          <scan>
-            <horizontal>
-              <samples>1</samples>
-              <resolution>1</resolution>
-              <min_angle>0</min_angle>
-              <max_angle>0</max_angle>
-            </horizontal>
-          </scan>
-          <range>
-            <min>0.01</min>
-            <max>0.04</max>
+        <visualize>true</visualize>
+        <ray>
+          <scan>
+            <horizontal>
+               <samples>720</samples>
+              <resolution>1</resolution>
+              <min_angle>-1.570796</min_angle>
+              <max_angle>1.570796</max_angle>
+            </horizontal>
+          </scan>
+          <range>
+            <min>0.01</min>
+            <max>0.5</max>
             <resolution>0.1</resolution>
           </range>
@@ -166,17 +166,17 @@
         <update_rate>20.0</update_rate>
         <pose>0 0 0 0 0 0</pose>
-        <visualize>false</visualize>
-        <ray>
-          <scan>
-            <horizontal>
-              <samples>1</samples>
-              <resolution>1</resolution>
-              <min_angle>0</min_angle>
-              <max_angle>0</max_angle>
-            </horizontal>
-          </scan>
-          <range>
-            <min>0.01</min>
-            <max>0.04</max>
+        <visualize>true</visualize>
+        <ray>
+          <scan>
+            <horizontal>
+               <samples>720</samples>
+              <resolution>1</resolution>
+              <min_angle>-1.570796</min_angle>
+              <max_angle>1.570796</max_angle>
+            </horizontal>
+          </scan>
+          <range>
+            <min>0.01</min>
+            <max>0.5</max>
             <resolution>0.1</resolution>
           </range>
@@ -189,17 +189,17 @@
         <update_rate>20.0</update_rate>
         <pose>0 0 0 0 0 0</pose>
-        <visualize>false</visualize>
-        <ray>
-          <scan>
-            <horizontal>
-              <samples>1</samples>
-              <resolution>1</resolution>
-              <min_angle>0</min_angle>
-              <max_angle>0</max_angle>
-            </horizontal>
-          </scan>
-          <range>
-            <min>0.01</min>
-            <max>0.04</max>
+        <visualize>true</visualize>
+        <ray>
+          <scan>
+            <horizontal>
+               <samples>720</samples>
+              <resolution>1</resolution>
+              <min_angle>-1.570796</min_angle>
+              <max_angle>1.570796</max_angle>
+            </horizontal>
+          </scan>
+          <range>
+            <min>0.01</min>
+            <max>0.5</max>
             <resolution>0.1</resolution>
           </range>

File: src/turtlebot/turtlebot_description/urdf/sensors/asus_xtion_pro.urdf.xacro (robot description, xacro)
@@ -3,4 +3,5 @@
   <xacro:include filename="$(find turtlebot_description)/urdf/sensors/camera_gazebo.urdf.xacro"/>
   <xacro:include filename="$(find turtlebot_description)/urdf/sensors/laser_gazebo.urdf.xacro"/>
+  <xacro:include filename="$(find turtlebot_description)/urdf/sensors/bumper_gazebo.urdf.xacro"/>
   <!-- Xacro properties -->
   <xacro:property name="M_SCALE" value="0.001"/>
@@ -8,13 +9,46 @@
   <xacro:property name="asus_xtion_pro_depth_rel_rgb_py" value="0.0270" />
   <xacro:property name="asus_xtion_pro_cam_rel_rgb_py"   value="-0.0220" />
+  <xacro:property name="cam_px_" value="0.13" />
+	<xacro:property name="cam_pz_" value="0.2870" />
+	<xacro:property name="cam_or_" value="0" />
+	<xacro:property name="cam_op_" value="0" />
+	<xacro:property name="cam_oy_" value="0" />
   <!-- Parameterised in part by the values in turtlebot_properties.urdf.xacro -->
   <xacro:macro name="sensor_asus_xtion_pro" params="parent">
     <joint name="camera_rgb_joint" type="fixed">
-      <origin xyz="${cam_px} ${asus_xtion_pro_cam_py} ${cam_pz}"
-              rpy="${cam_or} ${cam_op} ${cam_oy}"/>
+      <origin xyz="${cam_px_} ${asus_xtion_pro_cam_py} ${cam_pz_}"
+              rpy="${cam_or_} ${cam_op_} ${cam_oy_}"/>
       <parent link="${parent}"/>
       <child link="camera_rgb_frame" />
     </joint>
     <link name="camera_rgb_frame"/>
+    <!-- Asus mount -->
+    <joint name="mount_asus_xtion_pro_joint" type="fixed">
+      <origin xyz="-0.02 -0.0205 -0.015" rpy="0 0 0"/>
+      <parent link="camera_rgb_frame"/>
+      <child link="mount_asus_xtion_pro_link"/>
+    </joint>
+    <link name="mount_asus_xtion_pro_link">
+      <visual>
+        <origin xyz="0 0 0" rpy="${-M_PI/2} 0 0"/>
+        <geometry>
+          <mesh filename="package://turtlebot_description/meshes/sensors/xtion_pro_stack.dae"/>
+        </geometry>
+      </visual>
+      <collision>
+        <origin xyz="0.0 0.0 0.0" rpy="0 0 0" />
+        <geometry>
+        <!-- <box size="0.0330 0.2760 0.0120"/> -->
+        <box size="0.0 0.0 0.0"/>
+      </geometry>
+      </collision>
+      <inertial>
+        <mass value="0.170" />
+        <origin xyz="0 0 0" />
+        <inertia ixx="0.001152600" ixy="0.0" ixz="0.0"
+                 iyy="0.000148934" iyz="0.0"
+                 izz="0.001154654" />
+      </inertial>
+    </link>
     <joint name="camera_rgb_optical_joint" type="fixed">
       <origin xyz="0 0 0" rpy="${-M_PI/2} 0 ${-M_PI/2}" />
@@ -66,32 +100,5 @@
     <turtlebot_sim_3dsensor/>
     <turtlebot_sim_laser/>
-    <!-- Asus mount -->
-    <joint name="mount_asus_xtion_pro_joint" type="fixed">
-      <origin xyz="-0.1024 0.0 0.272" rpy="0 0 0"/>
-      <parent link="${parent}"/>
-      <child link="mount_asus_xtion_pro_link"/>
-    </joint>
-    <link name="mount_asus_xtion_pro_link">
-      <visual>
-        <origin xyz="0 0 0" rpy="${-M_PI/2} 0 0"/>
-        <geometry>
-          <mesh filename="package://turtlebot_description/meshes/sensors/xtion_pro_stack.dae"/>
-        </geometry>
-      </visual>
-      <collision>
-        <origin xyz="0.0 0.0 0.0" rpy="0 0 0" />
-        <geometry>
-        <!-- <box size="0.0330 0.2760 0.0120"/> -->
-        <box size="0.0 0.0 0.0"/>
-      </geometry>
-      </collision>
-      <inertial>
-        <mass value="0.170" />
-        <origin xyz="0 0 0" />
-        <inertia ixx="0.001152600" ixy="0.0" ixz="0.0"
-                 iyy="0.000148934" iyz="0.0"
-                 izz="0.001154654" />
-      </inertial>
-    </link>
+    <turtlebot_sim_bumper/>
   </xacro:macro>
 </robot>

File: src/turtlebot/turtlebot_description/urdf/stacks/circles.urdf.xacro (robot description, xacro)
@@ -80,5 +80,5 @@
         <origin xyz="0.0 0.0 0.0" rpy="0 0 0" />
         <geometry>
-          <cylinder length="0.0635" radius="0.0381"/>
+          <cylinder length="0.0635" radius="0.011"/>
         </geometry>
       </collision>
@@ -108,5 +108,5 @@
         <origin xyz="0.0 0.0 0.0" rpy="0 0 0" />
         <geometry>
-          <cylinder length="0.2032" radius="0.011113"/>
+          <cylinder length="0.3832" radius="0.011"/>
         </geometry>
       </collision>
@@ -134,7 +134,7 @@
       </visual>
       <collision>
-        <origin xyz="0.0 0.0 0.0" rpy="0 0 0" />
-        <geometry>
-          <cylinder length="0.008585" radius="0.001111"/>
+        <origin xyz="0.0 0.0 0.04" rpy="0 0 0" />
+        <geometry>
+          <cylinder length="0.08" radius="0.011"/>
         </geometry>
       </collision>
@@ -166,7 +166,8 @@
       </visual>
       <collision>
-        <origin xyz="0.0 0.0 0.0" rpy="0 0 0" />
-        <geometry>
-          <box size="0.233502 0.314845 0.006401"/>
+        <origin xyz="0.04334 0.0 0.0" rpy="0 0 0" />
+        <geometry>
+          <cylinder length="0.0064" radius="0.162"/>
+          <!-- <box size="0.233502 0.314845 0.006401"/> -->
           <!-- <box size="0.0 0.0 0.0"/> -->
         </geometry>
@@ -199,5 +200,6 @@
         <origin xyz="0.0 0.0 0.0" rpy="0 0 0" />
         <geometry>
-          <box size="0.314856 0.314856 0.006401"/>
+          <cylinder length="0.0064" radius="0.162"/>
+          <!-- <box size="0.314856 0.314856 0.006401"/> -->
           <!-- <box size="0.0 0.0 0.0"/> -->
         </geometry>
@@ -230,11 +232,11 @@
         <origin xyz="0.0 0.0 0.0" rpy="0 0 0" />
         <geometry>
-          <box size="0.314856 0.314856 0.006401"/>
+          <cylinder length="0.0064" radius="0.162"/>
           <!-- <box size="0.0 0.0 0.0"/> -->
         </geometry>
       </collision>
     </link>
-    <turtlebot_standoff_kinect parent="plate_2_link" number="0" x_loc="-0.1024382" y_loc="0.098" z_loc="0.0032004"/>
-    <turtlebot_standoff_kinect parent="plate_2_link" number="1" x_loc="-0.1024382" y_loc="-0.098" z_loc="0.0032004"/>
+    <turtlebot_standoff_kinect parent="plate_2_link" number="0" x_loc="0.11" y_loc="0.098" z_loc="0.0032004"/>
+    <turtlebot_standoff_kinect parent="plate_2_link" number="1" x_loc="0.11" y_loc="-0.098" z_loc="0.0032004"/>
     <turtlebot_standoff_8in parent="standoff_2in_4_link" number="0" x_loc="0" y_loc="0" z_loc="0.05715"/>
     <turtlebot_standoff_8in parent="standoff_2in_5_link" number="1" x_loc="0" y_loc="0" z_loc="0.05715"/>
@@ -261,8 +263,9 @@
       </visual>
       <collision>
-        <origin xyz="0.0 0.0 0.0" rpy="0 0 0" />
+        <origin xyz="0.01316 0.0 0.0" rpy="0 0 0" />
         <geometry>
           <!-- <box size="0.288 0.315 0.006401" /> -->
-          <box size="0.01 0.01 0.01" />
+          <!-- <box size="0.01 0.01 0.01" /> -->
+          <cylinder length="0.0064" radius="0.162"/>
         </geometry>
       </collision>

File: src/turtlebot/turtlebot_description/urdf/turtlebot_library.urdf.xacro (robot description, xacro)
@@ -17,3 +17,4 @@
   <xacro:include filename="$(find turtlebot_description)/urdf/sensors/asus_xtion_pro.urdf.xacro"/>
   <xacro:include filename="$(find turtlebot_description)/urdf/sensors/asus_xtion_pro_offset.urdf.xacro"/>
+  <xacro:include filename="$(find turtlebot_description)/urdf/sensors/realsense_d435.urdf.xacro"/>
 </robot>
