Commit message: update turtlebot show

File: src/turtlebot/turtlebot_description/urdf/bases/create.urdf.xacro (robot description, xacro)
@@ -2,5 +2,5 @@
 <robot name="turtlebot_hardware" xmlns:xacro="http://ros.org/wiki/xacro">
 	<!-- Macro for TurtleBot body. Including Gazebo extensions, but does not include Kinect -->
-		<xacro:include filename="$(find turtlebot_description)/urdf/bases/create_gazebo.urdf.xacro"/>
+	<xacro:include filename="$(find turtlebot_description)/urdf/bases/create_gazebo.urdf.xacro"/>
 	<!-- <xacro:property name="base_x" value="0.33" />
 	<xacro:property name="base_y" value="0.33" /> -->

File: src/turtlebot/turtlebot_description/urdf/bases/create_gazebo.urdf.xacro (robot description, xacro)
@@ -8,6 +8,7 @@
         <leftJoint>right_wheel_joint</leftJoint>
             <rightJoint>left_wheel_joint</rightJoint>
-        <wheelSeparation>.230</wheelSeparation>
-        <wheelDiameter>0.60</wheelDiameter>
+        <wheelSeparation>0.26</wheelSeparation>
+        <!-- <wheelDiameter>0.60</wheelDiameter> -->
+        <wheelDiameter>0.066</wheelDiameter>
         <torque>1.0</torque>
         <commandTopic>cmd_vel</commandTopic>
@@ -207,36 +208,4 @@
       </sensor>
 	  </gazebo>
-<!--
-    <gazebo reference="laser_sensor_link">
-      <sensor type="ray" name="laser_sensor">
-        <pose>0 0 0 0 0 0</pose>
-        <visualize>true</visualize>
-        <update_rate>40</update_rate>
-        <ray>
-          <scan>
-            <horizontal>
-              <samples>720</samples>
-              <resolution>1</resolution>
-              <min_angle>-1.570796</min_angle>
-              <max_angle>1.570796</max_angle>
-            </horizontal>
-          </scan>
-          <range>
-            <min>0.10</min>
-            <max>30.0</max>
-            <resolution>0.01</resolution>
-          </range>
-          <noise>
-            <type>gaussian</type>
-            <mean>0.0</mean>
-            <stddev>0.01</stddev>
-          </noise>
-        </ray>
-        <plugin name="gazebo_ros_head_hokuyo_controller" filename="libgazebo_ros_laser.so">
-          <topicName>/kobuki/laser/scan</topicName>
-          <frameName>laser_sensor_link</frameName>
-        </plugin>
-      </sensor>
-    </gazebo> -->
 	</xacro:macro>
 </robot>

File: src/turtlebot/turtlebot_description/urdf/obstacle.urdf.xacro (robot description, xacro)
@@ -4,233 +4,159 @@
 	<xacro:property name="obs_hight" value="1.6" />
 	<xacro:property name="obs_offset" value="0.83" />
-	<material name="Green"><color rgba="0.0 0.8 0.0 1.0"/></material>
-  	<material name="black"><color rgba="0.0 0.0 0.0 1.0" /></material>
-	<xacro:macro name="obstacle">
-		<gazebo>
-			<plugin name="differential_drive_controller" filename="libgazebo_ros_diff_drive.so">
-				<alwaysOn>true</alwaysOn>
-				<updateRate>50</updateRate>
-				<leftJoint>right_wheel_joint</leftJoint>
-				<rightJoint>left_wheel_joint</rightJoint>
-				<wheelSeparation>0.45</wheelSeparation>
-				<wheelDiameter>0.60</wheelDiameter>
-				<torque>1.0</torque>
-				<commandTopic>cmd_vel</commandTopic>
-				<odometryTopic>odom</odometryTopic>
-				<odometryFrame>odom</odometryFrame>
-				<robotBaseFrame>base_footprint</robotBaseFrame>
-				<publishWheelJointState>true</publishWheelJointState>
-				<legacyMode>true</legacyMode>
-				<rosDebugLevel>na</rosDebugLevel>
-				<publishWheelTF>false</publishWheelTF>
-				<wheelAcceleration>0</wheelAcceleration>
-				<wheelTorque>5</wheelTorque>
-				<odometrySource>world</odometrySource>
-				<publishTf>1</publishTf>
-			</plugin>
-		</gazebo>
-		<link name="obstacle_link">
-			<static>1</static>
-			<inertial>
-				<mass value="2" />
-				<origin xyz="0 0 0.0" />
-				<inertia ixx="0.01" ixy="0.0" ixz="0.0"
-					iyy="0.01" iyz="0.0" izz="0.5" />
-			</inertial>
-			<visual name='visual'>
-				<origin xyz="0 0 0" rpy="0 0 0" />
-				<geometry>
-					<cylinder radius="${obs_width}" length = "${obs_hight}"/>
-				</geometry>
-				<material name="black" />
-			</visual>
-			<collision name='collision'>
-				<origin xyz="0 0 0" rpy="0 0 0" />
-				<geometry>
-					<cylinder radius="${obs_width}" length = "${obs_hight}"/>
-				</geometry>
-			</collision>
-		</link>
-		<joint name="obstacle_joint" type="fixed">
-			<origin xyz="0 0 ${obs_offset}" rpy="0 0 0"/>
-			<parent link="base_link"/>
-			<child link="obstacle_link"/>
-		</joint>
-<!--
-		<link name="base_footprint">
-			<visual>
-				<origin xyz="0 0 0" rpy="0 0 0" />
-				<geometry>
-					<box size="0.001 0.001 0.001" />
-				</geometry>
-				<material name="Green" />
-			</visual>
-			<collision>
-				<origin xyz="0 0 0.017" rpy="0 0 0" />
-				<geometry>
-				<box size="0.001 0.001 0.001" />
-				</geometry>
-			</collision>
-		</link> -->
-		<link name="base_link">
-			<static>1</static>
-			<inertial>
-			<mass value="2" />
+  	<xacro:include filename="$(find turtlebot_description)/urdf/obstacle.gazebo" />
+	<xacro:include filename="$(find turtlebot_description)/urdf/materials.xacro" />
+	<link name="obstacle_link">
+		<static>1</static>
+		<collision name='collision'>
+			<origin xyz="0 0 0" rpy="0 0 0" />
+			<geometry>
+				<cylinder radius="${obs_width}" length = "${obs_hight}"/>
+			</geometry>
+		</collision>
+		<visual>
+			<origin xyz="0 0 0" rpy="0 0 0" />
+			<geometry>
+				<cylinder radius="${obs_width}" length = "${obs_hight}"/>
+			</geometry>
+			<material name="black"/>
+		</visual>
+		<inertial>
+			<mass value="0.02" />
 			<origin xyz="0 0 0.0" />
 			<inertia ixx="0.01" ixy="0.0" ixz="0.0"
 				iyy="0.01" iyz="0.0" izz="0.5" />
-			</inertial>
-			<visual>
-			<origin xyz=" 0 0 0.0308" rpy="0 0 0" />
+		</inertial>
+	</link>
+	<joint name="obstacle_joint" type="fixed">
+		<origin xyz="0 0 ${obs_offset}" rpy="0 0 0"/>
+		<parent link="base_link"/>
+		<child link="obstacle_link"/>
+	</joint>
+	<link name="base_link">
+		<static>1</static>
+		<inertial>
+		<mass value="2" />
+		<origin xyz="0 0 0.0" />
+		<inertia ixx="0.01" ixy="0.0" ixz="0.0"
+			iyy="0.01" iyz="0.0" izz="0.5" />
+		</inertial>
+		<visual>
+		<origin xyz=" 0 0 0.0308" rpy="0 0 0" />
+		<geometry>
+			<mesh filename="package://turtlebot_description/meshes/create_body.dae"/>
+		</geometry>
+		</visual>
+		<collision>
+		<origin xyz="0.0 0.0 0.0308" rpy="0 0 0" />
+		<geometry>
+			<cylinder length="0.0611632" radius="0.16495"/>
+		</geometry>
+		</collision>
+	</link>
+	<link name="left_wheel_link">
+		<inertial>
+		<origin xyz="0 0 0"/>
+		<mass value="0.01" />
+		<inertia ixx="0.001" ixy="0.0" ixz="0.0"
+			iyy="0.001" iyz="0.0" izz="0.001" />
+		</inertial>
+		<visual>
+		<origin xyz="0 0 0" rpy="0 1.5707 1.5707" />
+		<geometry>
+			<cylinder radius="0.033" length = "0.023"/>
+		</geometry>
+		</visual>
+		<collision>
+		<origin xyz="0 0 0" rpy="0 1.5707 1.5707" />
+		<geometry>
+			<cylinder radius="0.033" length = "0.023"/>
+		</geometry>
+		</collision>
+	</link>
+	<joint name="left_wheel_joint" type="continuous">
+		<origin xyz="0 0.13 0.015" rpy="0 0 0"/>
+		<parent link="base_link"/>
+		<child link="left_wheel_link"/>
+		<axis xyz="0 1 0"/>
+	</joint>
+	<link name="right_wheel_link">
+		<inertial>
+		<origin xyz="0 0 0"/>
+		<mass value="0.01" />
+		<inertia ixx="0.001" ixy="0.0" ixz="0.0"
+			iyy="0.001" iyz="0.0" izz="0.001" />
+		</inertial>
+		<visual>
+		<origin xyz="0 0 0" rpy="0 1.5707 1.5707" />
+		<geometry>
+			<cylinder radius="0.033" length = "0.023"/>
+		</geometry>
+		</visual>
+		<collision>
+		<origin xyz="0 0 0" rpy="0 1.5707 1.5707" />
+		<geometry>
+			<cylinder radius="0.033" length = "0.023"/>
+		</geometry>
+		</collision>
+	</link>
+	<joint name="right_wheel_joint" type="continuous">
+		<origin xyz="0 -0.13 0.015" rpy="0 0 0"/>
+		<parent link="base_link"/>
+		<child link="right_wheel_link"/>
+		<axis xyz="0 1 0"/>
+	</joint>
+	<link name="rear_wheel_link">
+		<inertial>
+			<origin xyz="0 0 0"/>
+			<mass value="0.001" />
+			<inertia ixx="0.0001" ixy="0.0" ixz="0.0"
+				iyy="0.0001" iyz="0.0" izz="0.0001" />
+		</inertial>
+		<visual>
+			<origin xyz="0 0 0" rpy="0 1.5707 1.5707"/>
 			<geometry>
-				<mesh filename="package://turtlebot_description/meshes/create_body.dae"/>
+				<sphere radius="0.015" />
 			</geometry>
-			</visual>
-			<collision>
-			<origin xyz="0.0 0.0 0.0308" rpy="0 0 0" />
+		</visual>
+		<collision>
+			<origin xyz="0 0 0" rpy="0 1.5707 1.5707" />
 			<geometry>
-				<cylinder length="0.0611632" radius="0.16495"/>
+				<sphere radius="0.015" />
 			</geometry>
-			</collision>
-		</link>
-		<link name="left_wheel_link">
-			<inertial>
-			<origin xyz="0 0 0"/>
+		</collision>
+	</link>
+	<!-- fixed because there's no transmission -->
+	<joint name="rear_castor_joint" type="fixed">
+		<origin xyz="-0.13 0 0.0" rpy="0 0 0"/>
+		<parent link="base_link"/>
+		<child link="rear_wheel_link"/>
+		<axis xyz="0 1 0"/>
+	</joint>
+	<link name="front_wheel_link">
+		<inertial>
+			<origin xyz="0 0 0" />
 			<mass value="0.01" />
 			<inertia ixx="0.001" ixy="0.0" ixz="0.0"
 				iyy="0.001" iyz="0.0" izz="0.001" />
-			</inertial>
-			<visual>
+		</inertial>
+		<visual>
+			<origin xyz="0 0 0" rpy="0 1.5707 1.5707"/>
+			<geometry>
+				<sphere radius="0.018" />
+			</geometry>
+		</visual>
+		<collision>
 			<origin xyz="0 0 0" rpy="0 1.5707 1.5707" />
 			<geometry>
-				<cylinder radius="0.033" length = "0.023"/>
+				<sphere radius="0.018" />
 			</geometry>
-			</visual>
-			<collision>
-			<origin xyz="0 0 0" rpy="0 1.5707 1.5707" />
-			<geometry>
-				<cylinder radius="0.033" length = "0.023"/>
-			</geometry>
-			</collision>
-		</link>
-		<joint name="left_wheel_joint" type="continuous">
-			<origin xyz="0 0.13 0.015" rpy="0 0 0"/>
-			<parent link="base_link"/>
-			<child link="left_wheel_link"/>
-			<axis xyz="0 1 0"/>
-		</joint>
-		<link name="right_wheel_link">
-			<inertial>
-			<origin xyz="0 0 0"/>
-			<mass value="0.01" />
-			<inertia ixx="0.001" ixy="0.0" ixz="0.0"
-				iyy="0.001" iyz="0.0" izz="0.001" />
-			</inertial>
-			<visual>
-			<origin xyz="0 0 0" rpy="0 1.5707 1.5707" />
-			<geometry>
-				<cylinder radius="0.033" length = "0.023"/>
-			</geometry>
-			</visual>
-			<collision>
-			<origin xyz="0 0 0" rpy="0 1.5707 1.5707" />
-			<geometry>
-				<cylinder radius="0.033" length = "0.023"/>
-			</geometry>
-			</collision>
-		</link>
-		<joint name="right_wheel_joint" type="continuous">
-			<origin xyz="0 -0.13 0.015" rpy="0 0 0"/>
-			<parent link="base_link"/>
-			<child link="right_wheel_link"/>
-			<axis xyz="0 1 0"/>
-		</joint>
-		<link name="rear_wheel_link">
-			<inertial>
-				<origin xyz="0 0 0"/>
-				<mass value="0.001" />
-				<inertia ixx="0.0001" ixy="0.0" ixz="0.0"
-					iyy="0.0001" iyz="0.0" izz="0.0001" />
-			</inertial>
-			<visual>
-				<origin xyz="0 0 0" rpy="0 1.5707 1.5707"/>
-				<geometry>
-					<sphere radius="0.015" />
-				</geometry>
-			</visual>
-			<collision>
-				<origin xyz="0 0 0" rpy="0 1.5707 1.5707" />
-				<geometry>
-					<sphere radius="0.015" />
-				</geometry>
-			</collision>
-		</link>
-		<!-- fixed because there's no transmission -->
-		<joint name="rear_castor_joint" type="fixed">
-			<origin xyz="-0.13 0 0.0" rpy="0 0 0"/>
-			<parent link="base_link"/>
-			<child link="rear_wheel_link"/>
-			<axis xyz="0 1 0"/>
-		</joint>
-		<link name="front_wheel_link">
-			<inertial>
-				<origin xyz="0 0 0" />
-				<mass value="0.01" />
-				<inertia ixx="0.001" ixy="0.0" ixz="0.0"
-					iyy="0.001" iyz="0.0" izz="0.001" />
-			</inertial>
-			<visual>
-				<origin xyz="0 0 0" rpy="0 1.5707 1.5707"/>
-				<geometry>
-					<sphere radius="0.018" />
-				</geometry>
-			</visual>
-			<collision>
-				<origin xyz="0 0 0" rpy="0 1.5707 1.5707" />
-				<geometry>
-					<sphere radius="0.018" />
-				</geometry>
-			</collision>
-		</link>
-		<!-- fixed because there's no transmission -->
-		<joint name="front_castor_joint" type="fixed">
-			<origin xyz="0.13 0 0.0" rpy="0 0 0"/>
-			<parent link="base_link"/>
-			<child link="front_wheel_link"/>
-			<axis xyz="0 1 0"/>
-		</joint>
-		<gazebo reference="left_wheel_link">
-		<mu1>1.0</mu1>
-		<mu2>1.0</mu2>
-		<kp>1000000.0</kp>
-		<kd>100.0</kd>
-		<minDepth>0.001</minDepth>
-		<maxVel>1.0</maxVel>
-		</gazebo>
-		<gazebo reference="right_wheel_link">
-		<mu1>1.0</mu1>
-		<mu2>1.0</mu2>
-		<kp>1000000.0</kp>
-		<kd>100.0</kd>
-		<minDepth>0.001</minDepth>
-		<maxVel>1.0</maxVel>
-		</gazebo>
-		<gazebo reference="rear_wheel_link">
-		<mu1>0.0</mu1>
-		<mu2>0.0</mu2>
-		<kp>1000000.0</kp>
-		<kd>100.0</kd>
-		<minDepth>0.001</minDepth>
-		<maxVel>1.0</maxVel>
-		</gazebo>
-		<gazebo reference="front_wheel_link">
-		<mu1>0.0</mu1>
-		<mu2>0.0</mu2>
-		<kp>1000000.0</kp>
-		<kd>100.0</kd>
-		<minDepth>0.001</minDepth>
-		<maxVel>1.0</maxVel>
-		</gazebo>
-  	</xacro:macro>
-	<obstacle/>
+		</collision>
+	</link>
+	<!-- fixed because there's no transmission -->
+	<joint name="front_castor_joint" type="fixed">
+		<origin xyz="0.13 0 0.0" rpy="0 0 0"/>
+		<parent link="base_link"/>
+		<child link="front_wheel_link"/>
+		<axis xyz="0 1 0"/>
+	</joint>
 </robot>

File: src/turtlebot/turtlebot_description/urdf/sensors/laser_gazebo.urdf.xacro (robot description, xacro)
@@ -4,5 +4,5 @@
   <xacro:macro name="turtlebot_sim_laser">
 	<gazebo reference="laser_sensor_link">
-		<sensor type="ray" name="laser_sensor">
+		<sensor type="gpu_ray" name="laser_sensor">
 			<pose>0 0 0 0 0 0</pose>
 			<visualize>true</visualize>
@@ -28,5 +28,5 @@
 				</noise>
 			</ray>
-			<plugin name="gazebo_ros_head_hokuyo_controller" filename="libgazebo_ros_laser.so">
+			<plugin name="gazebo_ros_head_hokuyo_controller" filename="libgazebo_ros_gpu_laser.so">
 				<topicName>/scan</topicName>
 				<frameName>laser_sensor_link</frameName>
