Commit message: add & fix obs_robot simulation

File: src/turtlebot/turtlebot_description/robots/create_circles_asus_xtion_pro.urdf.xacro (robot description, xacro)
@@ -3,5 +3,5 @@
     - Base      : create
     - Stacks    : circles
-    - 3d Sensor : kinect
+    - 3d Sensor : sensor_asus_xtion_pro
 -->
 <robot name="turtlebot" xmlns:xacro="http://ros.org/wiki/xacro">

File: src/turtlebot/turtlebot_description/robots/kobuki_hexagons_asus_xtion_pro.urdf.xacro (robot description, xacro)
@@ -3,5 +3,5 @@
     - Base      : kobuki
     - Stacks    : hexagons
-    - 3d Sensor : kinect
+    - 3d Sensor : sensor_asus_xtion_pro
 -->
 <robot name="turtlebot" xmlns:xacro="http://ros.org/wiki/xacro">

File: src/turtlebot/turtlebot_description/robots/kobuki_hexagons_asus_xtion_pro_offset.urdf.xacro (robot description, xacro)
@@ -3,5 +3,5 @@
     - Base      : kobuki
     - Stacks    : hexagons
-    - 3d Sensor : kinect
+    - 3d Sensor : sensor_asus_xtion_pro_offset
 -->
 <robot name="turtlebot" xmlns:xacro="http://ros.org/wiki/xacro">

File: src/turtlebot/turtlebot_description/urdf/bases/create.urdf.xacro (robot description, xacro)
@@ -1,18 +1,18 @@
 <?xml version="1.0"?>
 <robot name="turtlebot_hardware" xmlns:xacro="http://ros.org/wiki/xacro">
-  <!-- Macro for TurtleBot body. Including Gazebo extensions, but does not include Kinect -->
-  <xacro:include filename="$(find turtlebot_description)/urdf/bases/create_gazebo.urdf.xacro"/>
-  <xacro:property name="base_x" value="0.33" />
-  <xacro:property name="base_y" value="0.33" />
-	  <xacro:macro name="create">
-	    <material name="Green">
-	      <color rgba="0.0 0.8 0.0 1.0"/>
-	    </material>
-	  <joint name="laser_joint" type="fixed">
-	    <!-- <origin xyz="-0.065 0 0.075" rpy="0 0 0" /> -->
-		<origin xyz="0.0 0.0 0.42" rpy="0 0 0"/>
-	    <parent link="base_link" />
-	    <child link="laser_sensor_link" />
-	  </joint>
+	<!-- Macro for TurtleBot body. Including Gazebo extensions, but does not include Kinect -->
+		<xacro:include filename="$(find turtlebot_description)/urdf/bases/create_gazebo.urdf.xacro"/>
+	<!-- <xacro:property name="base_x" value="0.33" />
+	<xacro:property name="base_y" value="0.33" /> -->
+	<xacro:macro name="create">
+		<material name="Green">
+			<color rgba="0.0 0.8 0.0 1.0"/>
+		</material>
+		<joint name="laser_joint" type="fixed">
+			<!-- <origin xyz="-0.065 0 0.075" rpy="0 0 0" /> -->
+			<origin xyz="0.0 0.0 0.42" rpy="0 0 0"/>
+			<parent link="base_link" />
+			<child link="laser_sensor_link" />
+		</joint>
 		<link name="laser_sensor_link">
 			<inertial>
@@ -35,234 +35,234 @@
 			</visual>
 		</link>
-	  <!-- base_footprint is a fictitious link(frame) that is on the ground right below base_link origin, navigation stack depends on this frame -->
-	  <link name="base_footprint">
-	    <visual>
-	      <origin xyz="0 0 0" rpy="0 0 0" />
-	      <geometry>
-	        <box size="0.001 0.001 0.001" />
-	      </geometry>
-	      <material name="Green" />
-	    </visual>
-	    <collision>
-	      <origin xyz="0 0 0.017" rpy="0 0 0" />
-	      <geometry>
-	       <box size="0.001 0.001 0.001" />
-	      </geometry>
-	    </collision>
-	  </link>
-	  <link name="base_link">
-	    <inertial>
-	      <mass value="2" />
-	      <origin xyz="0 0 0.0" />
-	      <inertia ixx="0.01" ixy="0.0" ixz="0.0"
-	        iyy="0.01" iyz="0.0" izz="0.5" />
-	    </inertial>
-	    <visual>
-	      <origin xyz=" 0 0 0.0308" rpy="0 0 0" />
-	      <geometry>
-	        <mesh filename="package://turtlebot_description/meshes/create_body.dae"/>
-	      </geometry>
-	    </visual>
-	    <collision>
-	      <origin xyz="0.0 0.0 0.0308" rpy="0 0 0" />
-	      <geometry>
-	        <cylinder length="0.0611632" radius="0.16495"/>
-	      </geometry>
-	    </collision>
-	  </link>
-	  <link name="wall_sensor_link">
-	    <inertial>
-	      <mass value="0.01" />
-	      <origin xyz="0 0 0"/>
-	      <inertia ixx="0.001" ixy="0.0" ixz="0.0"
-	        iyy="0.001" iyz="0.0" izz="0.001" />
-	    </inertial>
-	  </link>
-	  <link name="left_cliff_sensor_link">
-	    <inertial>
-	      <mass value="0.01" />
-	      <origin xyz="0 0 0"/>
-	      <inertia ixx="0.001" ixy="0.0" ixz="0.0"
-	        iyy="0.001" iyz="0.0" izz="0.001" />
-	    </inertial>
-	  </link>
-	  <link name="right_cliff_sensor_link">
-	    <inertial>
-	      <mass value="0.01" />
-	      <origin xyz="0 0 0"/>
-	      <inertia ixx="0.001" ixy="0.0" ixz="0.0"
-	        iyy="0.001" iyz="0.0" izz="0.001" />
-	    </inertial>
-	  </link>
-	  <link name="leftfront_cliff_sensor_link">
-	    <inertial>
-	      <mass value="0.01" />
-	      <origin xyz="0 0 0"/>
-	      <inertia ixx="1.0" ixy="0.0" ixz="0.0"
-	        iyy="0.01" iyz="0.0" izz="0.01" />
-	    </inertial>
-	  </link>
-	  <link name="rightfront_cliff_sensor_link">
-	    <inertial>
-	      <mass value="0.01" />
-	      <origin xyz="0 0 0"/>
-	      <inertia ixx="0.001" ixy="0.0" ixz="0.0"
-	        iyy="0.001" iyz="0.0" izz="0.001" />
-	    </inertial>
-	  </link>
-	  <joint name="base_footprint_joint" type="fixed">
-	    <origin xyz="0 0 0.017" rpy="0 0 0" />
-	    <parent link="base_footprint"/>
-	    <child link="base_link" />
-	  </joint>
-	  <joint name="base_wall_sensor_joint" type="fixed">
-	    <origin xyz="0.09 -0.120 0.042" rpy="0 0 -1.0" />
-	    <parent link="base_link"/>
-	    <child link="wall_sensor_link" />
-	  </joint>
-	  <joint name="base_left_cliff_sensor_joint" type="fixed">
-	    <origin xyz="0.07 0.14 0.01" rpy="0 1.57079 0" />
-	    <parent link="base_link"/>
-	    <child link="left_cliff_sensor_link" />
-	  </joint>
-	  <joint name="base_right_cliff_sensor_joint" type="fixed">
-	    <origin xyz="0.07 -0.14 0.01" rpy="0 1.57079 0" />
-	    <parent link="base_link"/>
-	    <child link="right_cliff_sensor_link" />
-	  </joint>
-	  <joint name="base_leftfront_cliff_sensor_joint" type="fixed">
-	    <origin xyz="0.15 0.04 0.01" rpy="0 1.57079 0" />
-	    <parent link="base_link"/>
-	    <child link="leftfront_cliff_sensor_link" />
-	  </joint>
-	  <joint name="base_rightfront_cliff_sensor_joint" type="fixed">
-	    <origin xyz="0.15 -0.04 0.01" rpy="0 1.57079 0" />
-	    <parent link="base_link"/>
-	    <child link="rightfront_cliff_sensor_link" />
-	  </joint>
-	  <link name="left_wheel_link">
-	    <inertial>
-	      <origin xyz="0 0 0"/>
-	      <mass value="0.01" />
-	      <inertia ixx="0.001" ixy="0.0" ixz="0.0"
-	        iyy="0.001" iyz="0.0" izz="0.001" />
-	    </inertial>
-	    <visual>
-	      <origin xyz="0 0 0" rpy="0 1.5707 1.5707" />
-	      <geometry>
-	        <cylinder radius="0.033" length = "0.023"/>
-	      </geometry>
-	    </visual>
-	    <collision>
-	      <origin xyz="0 0 0" rpy="0 1.5707 1.5707" />
-	      <geometry>
-	        <cylinder radius="0.033" length = "0.023"/>
-	      </geometry>
-	    </collision>
-	  </link>
-	  <joint name="left_wheel_joint" type="continuous">
-	    <origin xyz="0 0.13 0.015" rpy="0 0 0"/>
-	    <parent link="base_link"/>
-	    <child link="left_wheel_link"/>
-	    <axis xyz="0 1 0"/>
-	  </joint>
-	  <link name="right_wheel_link">
-	    <inertial>
-	      <origin xyz="0 0 0"/>
-	      <mass value="0.01" />
-	      <inertia ixx="0.001" ixy="0.0" ixz="0.0"
-	        iyy="0.001" iyz="0.0" izz="0.001" />
-	    </inertial>
-	    <visual>
-	      <origin xyz="0 0 0" rpy="0 1.5707 1.5707" />
-	      <geometry>
-	        <cylinder radius="0.033" length = "0.023"/>
-	      </geometry>
-	    </visual>
-	    <collision>
-	      <origin xyz="0 0 0" rpy="0 1.5707 1.5707" />
-	      <geometry>
-	        <cylinder radius="0.033" length = "0.023"/>
-	      </geometry>
-	    </collision>
-	  </link>
-	  <joint name="right_wheel_joint" type="continuous">
-	    <origin xyz="0 -0.13 0.015" rpy="0 0 0"/>
-	    <parent link="base_link"/>
-	    <child link="right_wheel_link"/>
-	    <axis xyz="0 1 0"/>
-	  </joint>
-	  <link name="rear_wheel_link">
-	    <inertial>
-	      <origin xyz="0 0 0"/>
-	      <mass value="0.001" />
-	      <inertia ixx="0.0001" ixy="0.0" ixz="0.0"
-	        iyy="0.0001" iyz="0.0" izz="0.0001" />
-	    </inertial>
-	    <visual>
-	      <origin xyz="0 0 0" rpy="0 1.5707 1.5707"/>
-	      <geometry>
-	        <sphere radius="0.015" />
-	      </geometry>
-	    </visual>
-	    <collision>
-	      <origin xyz="0 0 0" rpy="0 1.5707 1.5707" />
-	      <geometry>
-	        <sphere radius="0.015" />
-	      </geometry>
-	    </collision>
-	  </link>
-	  <!-- fixed because there's no transmission -->
-	  <joint name="rear_castor_joint" type="fixed">
-	    <origin xyz="-0.13 0 0.0" rpy="0 0 0"/>
-	    <parent link="base_link"/>
-	    <child link="rear_wheel_link"/>
-	    <axis xyz="0 1 0"/>
-	  </joint>
-	  <link name="front_wheel_link">
-	    <inertial>
-	      <origin xyz="0 0 0" />
-	      <mass value="0.01" />
-	      <inertia ixx="0.001" ixy="0.0" ixz="0.0"
-	        iyy="0.001" iyz="0.0" izz="0.001" />
-	    </inertial>
-	    <visual>
-	      <origin xyz="0 0 0" rpy="0 1.5707 1.5707"/>
-	      <geometry>
-	        <sphere radius="0.018" />
-	      </geometry>
-	    </visual>
-	    <collision>
-	      <origin xyz="0 0 0" rpy="0 1.5707 1.5707" />
-	      <geometry>
-	        <sphere radius="0.018" />
-	      </geometry>
-	    </collision>
-	  </link>
-	  <!-- fixed because there's no transmission -->
-	  <joint name="front_castor_joint" type="fixed">
-	    <origin xyz="0.13 0 0.0" rpy="0 0 0"/>
-	    <parent link="base_link"/>
-	    <child link="front_wheel_link"/>
-	    <axis xyz="0 1 0"/>
-	  </joint>
-	  <joint name="gyro_joint" type="fixed">
-	    <axis xyz="0 1 0" />
-	    <origin xyz="0 0 0.04" rpy="0 0 0" />
-	    <parent link="base_link"/>
-	    <child link="gyro_link"/>
-	  </joint>
-	  <link name="gyro_link">
-	    <inertial>
-	      <mass value="0.001" />
-	      <origin xyz="0 0 0" rpy="0 0 0" />
-	      <inertia ixx="0.0001" ixy="0" ixz="0" iyy="0.000001" iyz="0" izz="0.0001" />
-	    </inertial>
-	  </link>
+		<!-- base_footprint is a fictitious link(frame) that is on the ground right below base_link origin, navigation stack depends on this frame -->
+		<link name="base_footprint">
+			<visual>
+			<origin xyz="0 0 0" rpy="0 0 0" />
+			<geometry>
+				<box size="0.001 0.001 0.001" />
+			</geometry>
+			<material name="Green" />
+			</visual>
+			<collision>
+			<origin xyz="0 0 0.017" rpy="0 0 0" />
+			<geometry>
+			<box size="0.001 0.001 0.001" />
+			</geometry>
+			</collision>
+		</link>
+		<link name="base_link">
+			<inertial>
+			<mass value="2" />
+			<origin xyz="0 0 0.0" />
+			<inertia ixx="0.01" ixy="0.0" ixz="0.0"
+				iyy="0.01" iyz="0.0" izz="0.5" />
+			</inertial>
+			<visual>
+			<origin xyz=" 0 0 0.0308" rpy="0 0 0" />
+			<geometry>
+				<mesh filename="package://turtlebot_description/meshes/create_body.dae"/>
+			</geometry>
+			</visual>
+			<collision>
+			<origin xyz="0.0 0.0 0.0308" rpy="0 0 0" />
+			<geometry>
+				<cylinder length="0.0611632" radius="0.16495"/>
+			</geometry>
+			</collision>
+		</link>
+		<link name="left_wheel_link">
+			<inertial>
+			<origin xyz="0 0 0"/>
+			<mass value="0.01" />
+			<inertia ixx="0.001" ixy="0.0" ixz="0.0"
+				iyy="0.001" iyz="0.0" izz="0.001" />
+			</inertial>
+			<visual>
+			<origin xyz="0 0 0" rpy="0 1.5707 1.5707" />
+			<geometry>
+				<cylinder radius="0.033" length = "0.023"/>
+			</geometry>
+			</visual>
+			<collision>
+			<origin xyz="0 0 0" rpy="0 1.5707 1.5707" />
+			<geometry>
+				<cylinder radius="0.033" length = "0.023"/>
+			</geometry>
+			</collision>
+		</link>
+		<joint name="left_wheel_joint" type="continuous">
+			<origin xyz="0 0.13 0.015" rpy="0 0 0"/>
+			<parent link="base_link"/>
+			<child link="left_wheel_link"/>
+			<axis xyz="0 1 0"/>
+		</joint>
+		<link name="right_wheel_link">
+			<inertial>
+			<origin xyz="0 0 0"/>
+			<mass value="0.01" />
+			<inertia ixx="0.001" ixy="0.0" ixz="0.0"
+				iyy="0.001" iyz="0.0" izz="0.001" />
+			</inertial>
+			<visual>
+			<origin xyz="0 0 0" rpy="0 1.5707 1.5707" />
+			<geometry>
+				<cylinder radius="0.033" length = "0.023"/>
+			</geometry>
+			</visual>
+			<collision>
+			<origin xyz="0 0 0" rpy="0 1.5707 1.5707" />
+			<geometry>
+				<cylinder radius="0.033" length = "0.023"/>
+			</geometry>
+			</collision>
+		</link>
+		<joint name="right_wheel_joint" type="continuous">
+			<origin xyz="0 -0.13 0.015" rpy="0 0 0"/>
+			<parent link="base_link"/>
+			<child link="right_wheel_link"/>
+			<axis xyz="0 1 0"/>
+		</joint>
+		<link name="rear_wheel_link">
+			<inertial>
+				<origin xyz="0 0 0"/>
+				<mass value="0.001" />
+				<inertia ixx="0.0001" ixy="0.0" ixz="0.0"
+					iyy="0.0001" iyz="0.0" izz="0.0001" />
+			</inertial>
+			<visual>
+				<origin xyz="0 0 0" rpy="0 1.5707 1.5707"/>
+				<geometry>
+					<sphere radius="0.015" />
+				</geometry>
+			</visual>
+			<collision>
+				<origin xyz="0 0 0" rpy="0 1.5707 1.5707" />
+				<geometry>
+					<sphere radius="0.015" />
+				</geometry>
+			</collision>
+		</link>
+		<!-- fixed because there's no transmission -->
+		<joint name="rear_castor_joint" type="fixed">
+			<origin xyz="-0.13 0 0.0" rpy="0 0 0"/>
+			<parent link="base_link"/>
+			<child link="rear_wheel_link"/>
+			<axis xyz="0 1 0"/>
+		</joint>
+		<link name="front_wheel_link">
+			<inertial>
+				<origin xyz="0 0 0" />
+				<mass value="0.01" />
+				<inertia ixx="0.001" ixy="0.0" ixz="0.0"
+					iyy="0.001" iyz="0.0" izz="0.001" />
+			</inertial>
+			<visual>
+				<origin xyz="0 0 0" rpy="0 1.5707 1.5707"/>
+				<geometry>
+					<sphere radius="0.018" />
+				</geometry>
+			</visual>
+			<collision>
+				<origin xyz="0 0 0" rpy="0 1.5707 1.5707" />
+				<geometry>
+					<sphere radius="0.018" />
+				</geometry>
+			</collision>
+		</link>
+		<!-- fixed because there's no transmission -->
+		<joint name="front_castor_joint" type="fixed">
+			<origin xyz="0.13 0 0.0" rpy="0 0 0"/>
+			<parent link="base_link"/>
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
File: src/turtlebot/turtlebot_description/urdf/bases/create_gazebo.urdf.xacro (robot description, xacro)
@@ -2,27 +2,27 @@
 <robot xmlns:xacro="http://ros.org/wiki/xacro" name="turtlebot_gazebo">
 	<xacro:macro name="sim_create">
-   <gazebo>
+    <gazebo>
       <plugin name="differential_drive_controller" filename="libgazebo_ros_diff_drive.so">
-	    <alwaysOn>true</alwaysOn>
-	    <updateRate>50</updateRate>
-	    <leftJoint>right_wheel_joint</leftJoint>
-    	    <rightJoint>left_wheel_joint</rightJoint>
-	    <wheelSeparation>.230</wheelSeparation>
-	    <wheelDiameter>0.070</wheelDiameter>
-	    <torque>1.0</torque>
-	    <commandTopic>cmd_vel</commandTopic>
-	    <odometryTopic>odom</odometryTopic>
-	    <odometryFrame>odom</odometryFrame>
-	    <robotBaseFrame>base_footprint</robotBaseFrame>
-	    <publishWheelJointState>true</publishWheelJointState>
-	    <legacyMode>true</legacyMode>
-	    <rosDebugLevel>na</rosDebugLevel>
-	    <publishWheelTF>false</publishWheelTF>
-      <wheelAcceleration>0</wheelAcceleration>
-      <wheelTorque>5</wheelTorque>
-      <odometrySource>world</odometrySource>
-      <publishTf>1</publishTf>
-	  </plugin>
-	</gazebo>
+        <alwaysOn>true</alwaysOn>
+        <updateRate>50</updateRate>
+        <leftJoint>right_wheel_joint</leftJoint>
+            <rightJoint>left_wheel_joint</rightJoint>
+        <wheelSeparation>.230</wheelSeparation>
+        <wheelDiameter>0.070</wheelDiameter>
+        <torque>1.0</torque>
+        <commandTopic>cmd_vel</commandTopic>
+        <odometryTopic>odom</odometryTopic>
+        <odometryFrame>odom</odometryFrame>
+        <robotBaseFrame>base_footprint</robotBaseFrame>
+        <publishWheelJointState>true</publishWheelJointState>
+        <legacyMode>true</legacyMode>
+        <rosDebugLevel>na</rosDebugLevel>
+        <publishWheelTF>false</publishWheelTF>
+        <wheelAcceleration>0</wheelAcceleration>
+        <wheelTorque>5</wheelTorque>
+        <odometrySource>world</odometrySource>
+        <publishTf>1</publishTf>
+      </plugin>
+    </gazebo>
 <!--
 	  <gazebo>

File: src/turtlebot/turtlebot_description/urdf/stacks/circles.urdf.xacro (robot description, xacro)
@@ -263,5 +263,4 @@
         <origin xyz="0.0 0.0 0.0" rpy="0 0 0" />
         <geometry>
-          <!-- 原尺寸阻挡激光 -->
           <!-- <box size="0.288 0.315 0.006401" /> -->
           <box size="0.01 0.01 0.01" />
