Commit message: add random init position for obs

File: src/turtlebot/turtlebot_description/urdf/obstacle.urdf.xacro (robot description, xacro)
@@ -31,12 +31,12 @@
 		</gazebo>
 		<link name="obstacle_link">
-			<!-- <static>1</static> -->
-			<!-- <inertial>
+			<static>1</static>
+			<inertial>
 				<mass value="2" />
 				<origin xyz="0 0 0.0" />
 				<inertia ixx="0.01" ixy="0.0" ixz="0.0"
 					iyy="0.01" iyz="0.0" izz="0.5" />
-			</inertial> -->
-			<visual>
+			</inertial>
+			<visual name='visual'>
 				<origin xyz="0 0 0" rpy="0 0 0" />
 				<geometry>
@@ -45,8 +45,8 @@
 				<material name="black" />
 			</visual>
-			<collision>
+			<collision name='collision'>
 				<origin xyz="0 0 0" rpy="0 0 0" />
 				<geometry>
-					<cylinder radius="${obs_width}" length = "${obs_width}"/>
+					<cylinder radius="${obs_width}" length = "${obs_hight}"/>
 				</geometry>
 			</collision>
@@ -74,4 +74,5 @@
 		</link> -->
 		<link name="base_link">
+			<static>1</static>
 			<inertial>
 			<mass value="2" />

Commit message: :rocket:UPDATE

File: src/turtlebot/turtlebot_description/urdf/obstacle.urdf.xacro (robot description, xacro)
@@ -2,10 +2,16 @@
 <robot name="obstacle" xmlns:xacro="http://ros.org/wiki/xacro">
 	<xacro:property name="obs_width" value="0.25" />
-	<xacro:property name="obs_hight" value="1.6" />
-	<xacro:property name="obs_offset" value="0.83" />
+	<xacro:property name="obs_hight" value="1.0" />
+	<xacro:property name="obs_offset" value="0.53" />
   	<xacro:include filename="$(find turtlebot_description)/urdf/obstacle.gazebo" />
 	<xacro:include filename="$(find turtlebot_description)/urdf/materials.xacro" />
 	<link name="obstacle_link">
 		<static>1</static>
+		<inertial>
+			<mass value="0.2" />
+			<origin xyz="0 0 0.0" />
+			<inertia ixx="0.01" ixy="0.0" ixz="0.0"
+				iyy="0.01" iyz="0.0" izz="0.5" />
+		</inertial>
 		<collision name='collision'>
 			<origin xyz="0 0 0" rpy="0 0 0" />
@@ -21,10 +27,4 @@
 			<material name="black"/>
 		</visual>
-		<inertial>
-			<mass value="0.02" />
-			<origin xyz="0 0 0.0" />
-			<inertia ixx="0.01" ixy="0.0" ixz="0.0"
-				iyy="0.01" iyz="0.0" izz="0.5" />
-		</inertial>
 	</link>
 	<joint name="obstacle_joint" type="fixed">
@@ -36,8 +36,8 @@
 		<static>1</static>
 		<inertial>
-		<mass value="2" />
-		<origin xyz="0 0 0.0" />
-		<inertia ixx="0.01" ixy="0.0" ixz="0.0"
-			iyy="0.01" iyz="0.0" izz="0.5" />
+			<mass value="2" />
+			<origin xyz="0 0 0.0" />
+			<inertia ixx="0.01" ixy="0.0" ixz="0.0"
+				iyy="0.01" iyz="0.0" izz="0.5" />
 		</inertial>
 		<visual>

File: src/turtlebot/turtlebot_description/urdf/sensors/bumper_gazebo.urdf.xacro (robot description, xacro)
@@ -6,5 +6,5 @@
                 <visualize>true</visualize>
                 <always_on>true</always_on>
-                <update_rate>50.0</update_rate>
+                <update_rate>120.0</update_rate>
                 <contact>
                     <collision>base_footprint_fixed_joint_lump__base_link_collision_1</collision>
@@ -12,5 +12,5 @@
                 <plugin name="gazebo_ros_bumper_controller" filename="libgazebo_ros_bumper.so">
                     <alwaysOn>true</alwaysOn>
-                    <updateRate>50.0</updateRate>
+                    <updateRate>120.0</updateRate>
                     <bumperTopicName>base_bumper</bumperTopicName>
                     <frameName>base_link</frameName>

File: src/turtlebot/turtlebot_description/urdf/sensors/camera_gazebo.urdf.xacro (robot description, xacro)
@@ -6,5 +6,5 @@
       <sensor type="depth" name="camera">
         <always_on>true</always_on>
-        <update_rate>60.0</update_rate>
+        <update_rate>120.0</update_rate>
         <camera>
           <horizontal_fov>${60.0*M_PI/180.0}</horizontal_fov>
@@ -22,5 +22,5 @@
           <cameraName>camera</cameraName>
           <alwaysOn>true</alwaysOn>
-          <updateRate>60</updateRate>
+          <updateRate>120</updateRate>
           <imageTopicName>rgb/image_raw</imageTopicName>
           <depthImageTopicName>depth/image_raw</depthImageTopicName>

File: src/turtlebot/turtlebot_description/urdf/sensors/laser_gazebo.urdf.xacro (robot description, xacro)
@@ -6,18 +6,20 @@
 		<sensor type="gpu_ray" name="laser_sensor">
 			<pose>0 0 0 0 0 0</pose>
-			<visualize>true</visualize>
+			<visualize>False</visualize>
 			<update_rate>50</update_rate>
 			<ray>
 				<scan>
 					<horizontal>
-						<samples>720</samples>
+						<samples>90</samples>
 						<resolution>1</resolution>
-						<min_angle>-${M_PI}</min_angle>
-						<max_angle>${M_PI}</max_angle>
+						<!-- <min_angle>-${M_PI}</min_angle>
+						<max_angle>${M_PI}</max_angle> -->
+						<min_angle>-${M_PI/4}</min_angle>
+						<max_angle>${M_PI/4}</max_angle>
 					</horizontal>
 				</scan>
 				<range>
 					<min>0.10</min>
-					<max>10.0</max>
+					<max>3.0</max>
 					<resolution>0.01</resolution>
 				</range>
